File: kicad/_autosave-stepper_monitor.kicad_pcb (KiCad board)
At the start: 2 copper layers, 53 parts, among them J1 USB_C_Receptacle_USB2.0, J2 Conn_01x02_Male, J3 JTAG, J4 Conn_01x04_Male, J5 Conn_01x04_Male, Q1 UMH3N, Q2 PJA3439, Q3 AO3416, SW1 SW_Push, U1 CP2102N-A01-GQFN28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

Commit message: Updated the schematic: Fixed the power selection circuit.
Parts:
- removed Q3: AO3416, Package_TO_SOT_SMD:SOT-23
- added J6: Conn_01x03_Male, Connector_PinHeader_2.54mm:PinHeader_1x03_P2.54mm_Vertical, F.Cu at (55.9, 77.5)
- moved D5 90.7 mm to (77.5, 110.5)
- moved R7 81.4 mm to (74.9, 55.9)
- moved Q1 66.4 mm to (78.7, 74.9)
- moved U2 2.84 mm to (81.3, 97.8)
Connections:
- C10 pad 2: Net-(C1-Pad2) -> Net-(C10-Pad2)
- C9 pad 2: Net-(C1-Pad2) -> Net-(C10-Pad2)
- U4 pad 3: Net-(C1-Pad2) -> Net-(C10-Pad2)
Changed lines of the file:
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@@
   (net 87 "CFG2")
   (net 88 "SWITCH")
+  (net 89 "Net-(C10-Pad2)")
   (footprint "Capacitor_SMD:C_0402_1005Metric" (layer "F.Cu")
     (at 130.937 79.629)
@@
     )
   )
+  (footprint "Connector_PinHeader_2.54mm:PinHeader_1x03_P2.54mm_Vertical" (layer "F.Cu")
+    (at 55.88 77.47)
+    (descr "Through hole straight pin header, 1x03, 2.54mm pitch, single row")
+    (tags "Through hole pin header THT 1x03 2.54mm single row")
+    (property "Sheetfile" "stepper_monitor.kicad_sch")
+    (property "Sheetname" "")
+    (attr through_hole)
+    (fp_text reference "J6" (at 0 -2.33) (layer "F.SilkS")
+      (effects (font (size 1 1) (thickness 0.15)))
+    )
+    (fp_text value "Conn_01x03_Male" (at 0 7.41) (layer "F.Fab")
+      (effects (font (size 1 1) (thickness 0.15)))
+    )
+    (fp_text user "${REFERENCE}" (at 0 2.54 90) (layer "F.Fab")
+      (effects (font (size 1 1) (thickness 0.15)))
+    )
+    (fp_line (start 1.33 1.27) (end 1.33 6.41) (layer "F.SilkS") (width 0.12))
+    (fp_line (start -1.33 1.27) (end 1.33 1.27) (layer "F.SilkS") (width 0.12))
+    (fp_line (start -1.33 6.41) (end 1.33 6.41) (layer "F.SilkS") (width 0.12))
+    (fp_line (start -1.33 -1.33) (end 0 -1.33) (layer "F.SilkS") (width 0.12))
+    (fp_line (start -1.33 0) (end -1.33 -1.33) (layer "F.SilkS") (width 0.12))
+    (fp_line (start -1.33 1.27) (end -1.33 6.41) (layer "F.SilkS") (width 0.12))
+    (fp_line (start 1.8 6.85) (end 1.8 -1.8) (layer "F.CrtYd") (width 0.05))
+    (fp_line (start -1.8 6.85) (end 1.8 6.85) (layer "F.CrtYd") (width 0.05))
+    (fp_line (start -1.8 -1.8) (end -1.8 6.85) (layer "F.CrtYd") (width 0.05))
+    (fp_line (start 1.8 -1.8) (end -1.8 -1.8) (layer "F.CrtYd") (width 0.05))
+    (fp_line (start -1.27 -0.635) (end -0.635 -1.27) (layer "F.Fab") (width 0.1))
+    (fp_line (start -0.635 -1.27) (end 1.27 -1.27) (layer "F.Fab") (width 0.1))
+    (fp_line (start 1.27 -1.27) (end 1.27 6.35) (layer "F.Fab") (width 0.1))
+    (fp_line (start 1.27 6.35) (end -1.27 6.35) (layer "F.Fab") (width 0.1))
+    (fp_line (start -1.27 6.35) (end -1.27 -0.635) (layer "F.Fab") (width 0.1))
+    (pad "1" thru_hole rect (at 0 0) (size 1.7 1.7) (drill 1) (layers *.Cu *.Mask)
+      (net 89 "Net-(C10-Pad2)") (pinfunction "Pin_1") (pintype "passive"))
+    (pad "2" thru_hole oval (at 0 2.54) (size 1.7 1.7) (drill 1) (layers *.Cu *.Mask)
+      (net 61 "Net-(C1-Pad2)") (pinfunction "Pin_2") (pintype "passive"))
+    (pad "3" thru_hole oval (at 0 5.08) (size 1.7 1.7) (drill 1) (layers *.Cu *.Mask)
+      (net 62 "VBUS") (pinfunction "Pin_3") (pintype "passive"))
+    (model "${KICAD6_3DMODEL_DIR}/Connector_PinHeader_2.54mm.3dshapes/PinHeader_1x03_P2.54mm_Vertical.wrl"
+      (offset (xyz 0 0 0))
+      (scale (xyz 1 1 1))
+      (rotate (xyz 0 0 0))
+    )
+  )
   (footprint "Resistor_SMD:R_0402_1005Metric" (layer "F.Cu")
     (at 179.21 73.58)
@@
   )
   (footprint "Package_TO_SOT_SMD:SOT-223-3_TabPin2" (layer "F.Cu")
-    (at 80.01 100.33 90)
+    (at 81.28 97.79 90)
     (descr "module CMS SOT223 4 pins")
     (tags "CMS SOT")
@@
   )
   (footprint "Package_TO_SOT_SMD:SOT-363_SC-70-6" (layer "F.Cu")
-    (at 139.95 100.55 -90)
+    (at 78.74 74.93 -90)
     (descr "SOT-363, SC-70-6")
     (tags "SOT-363 SC-70-6")
@@
       (net 17 "GNDD") (pinfunction "GND") (pintype "input"))
     (pad "3" smd rect (at 2.54 2.84 180) (size 1.25 4.12) (layers "F.Cu" "F.Paste" "F.Mask")
-      (net 61 "Net-(C1-Pad2)") (pinfunction "OUT") (pintype "power_out"))
+      (net 89 "Net-(C10-Pad2)") (pinfunction "OUT") (pintype "power_out"))
     (pad "4" smd rect (at 2.54 -3.49 180) (size 1.05 2.82) (layers "F.Cu" "F.Paste" "F.Mask")
       (net 53 "unconnected-(U4-Pad4)") (pintype "no_connect"))
@@
     )
   )
-  (footprint "Package_TO_SOT_SMD:SOT-23" (layer "F.Cu")
-    (at 171.45 90.17 90)
-    (descr "SOT, 3 Pin (https://www.jedec.org/system/files/docs/to-236h.pdf variant AB), generated with kicad-footprint-generator ipc_gullwing_generator.py")
-    (tags "SOT TO_SOT_SMD")
-    (property "LCSC" "C479060")
-    (property "Sheetfile" "stepper_monitor.kicad_sch")
-    (property "Sheetname" "")
-    (attr smd)
-    (fp_text reference "Q3" (at 0 -2.4 90) (layer "F.SilkS")
-      (effects (font (size 1 1) (thickness 0.15)))
-    )
-    (fp_text value "AO3416" (at 0 2.4 90) (layer "F.Fab")
-      (effects (font (size 1 1) (thickness 0.15)))
-    )
-    (fp_text user "${REFERENCE}" (at 0 0 90) (layer "F.Fab")
-      (effects (font (size 0.32 0.32) (thickness 0.05)))
-    )
-    (fp_line (start 0 1.56) (end 0.65 1.56) (layer "F.SilkS") (width 0.12))
-    (fp_line (start 0 1.56) (end -0.65 1.56) (layer "F.SilkS") (width 0.12))
-    (fp_line (start 0 -1.56) (end 0.65 -1.56) (layer "F.SilkS") (width 0.12))
-    (fp_line (start 0 -1.56) (end -1.675 -1.56) (layer "F.SilkS") (width 0.12))
-    (fp_line (start -1.92 -1.7) (end -1.92 1.7) (layer "F.CrtYd") (width 0.05))
-    (fp_line (start 1.92 -1.7) (end -1.92 -1.7) (layer "F.CrtYd") (width 0.05))
-    (fp_line (start 1.92 1.7) (end 1.92 -1.7) (layer "F.CrtYd") (width 0.05))
-    (fp_line (start -1.92 1.7) (end 1.92 1.7) (layer "F.CrtYd") (width 0.05))
-    (fp_line (start -0.325 -1.45) (end 0.65 -1.45) (layer "F.Fab") (width 0.1))
-    (fp_line (start -0.65 1.45) (end -0.65 -1.125) (layer "F.Fab") (width 0.1))
-    (fp_line (start 0.65 -1.45) (end 0.65 1.45) (layer "F.Fab") (width 0.1))
-    (fp_line (start 0.65 1.45) (end -0.65 1.45) (layer "F.Fab") (width 0.1))
-    (fp_line (start -0.65 -1.125) (end -0.325 -1.45) (layer "F.Fab") (width 0.1))
-    (pad "1" smd roundrect (at -0.9375 -0.95 90) (size 1.475 0.6) (layers "F.Cu" "F.Paste" "F.Mask") (roundrect_rratio 0.25)
-      (net 17 "GNDD") (pinfunction "G") (pintype "input"))
-    (pad "2" smd roundrect (at -0.9375 0.95 90) (size 1.475 0.6) (layers "F.Cu" "F.Paste" "F.Mask") (roundrect_rratio 0.25)
-      (net 61 "Net-(C1-Pad2)") (pinfunction "S") (pintype "passive"))
-    (pad "3" smd roundrect (at 0.9375 0 90) (size 1.475 0.6) (layers "F.Cu" "F.Paste" "F.Mask") (roundrect_rratio 0.25)
-      (net 62 "VBUS") (pinfunction "D") (pintype "passive"))
-    (model "${KICAD6_3DMODEL_DIR}/Package_TO_SOT_SMD.3dshapes/SOT-23.wrl"
-      (offset (xyz 0 0 0))
-      (scale (xyz 1 1 1))
-      (rotate (xyz 0 0 0))
-    )
-  )
   (footprint "Capacitor_SMD:C_0402_1005Metric" (layer "F.Cu")
     (at 179.44 77.55)
@@
       (net 17 "GNDD") (pintype "passive"))
     (pad "2" smd roundrect (at 0.48 0) (size 0.56 0.62) (layers "F.Cu" "F.Paste" "F.Mask") (roundrect_rratio 0.25)
-      (net 61 "Net-(C1-Pad2)") (pintype "passive"))
+      (net 89 "Net-(C10-Pad2)") (pintype "passive"))
     (model "${KICAD6_3DMODEL_DIR}/Capacitor_SMD.3dshapes/C_0402_1005Metric.wrl"
       (offset (xyz 0 0 0))
@@
   )
   (footprint "Resistor_SMD:R_0402_1005Metric" (layer "F.Cu")
-    (at 143.53 99.62)
+    (at 74.93 55.88)
     (descr "Resistor SMD 0402 (1005 Metric), square (rectangular) end terminal, IPC_7351 nominal, (Body size source: IPC-SM-782 page 72, https://www.pcb-3d.com/wordpress/wp-content/uploads/ipc-sm-782a_amendment_1_and_2.pdf), generated with kicad-footprint-generator")
     (tags "resistor")
@@
   )
   (footprint "stepper_probe:D_MiniMELF_zenner" (layer "F.Cu")
-    (at 160.83 74.71)
+    (at 77.47 110.49)
     (descr "Diode Mini-MELF (SOD-80)")
     (tags "Diode Mini-MELF (SOD-80)")
@@
       (net 17 "GNDD") (pintype "passive"))
     (pad "2" smd roundrect (at 0.48 0) (size 0.56 0.62) (layers "F.Cu" "F.Paste" "F.Mask") (roundrect_rratio 0.25)
-      (net 61 "Net-(C1-Pad2)") (pintype "passive"))
+      (net 89 "Net-(C10-Pad2)") (pintype "passive"))
     (model "${KICAD6_3DMODEL_DIR}/Capacitor_SMD.3dshapes/C_0402_1005Metric.wrl"
       (offset (xyz 0 0 0))
